Commit message: Немного изменений для более менее нормального контакта между схватом и кубиком

File: urdf/cube_red.urdf (robot description, URDF)
Before this commit: robot simple_box, 1 links, 0 joints
Links:
- link my_box: geometry collision box size=0.05 0.05 0.15; visual box size=0.05 0.05 0.15

File: urdf/ur5_joint_limited_robot.urdf.xacro (robot description, xacro)
@@ -9,7 +9,7 @@
   <!-- arm -->
   <xacro:ur5_robot prefix="" joint_limited="true"
-    shoulder_pan_lower_limit="${-2*pi}" shoulder_pan_upper_limit="${2*pi}"
-    shoulder_lift_lower_limit="${-2*pi}" shoulder_lift_upper_limit="${2*pi}"
-    elbow_joint_lower_limit="${-2*pi}" elbow_joint_upper_limit="${2*pi}"
+    shoulder_pan_lower_limit="${-pi}" shoulder_pan_upper_limit="${pi}"
+    shoulder_lift_lower_limit="${-pi}" shoulder_lift_upper_limit="${pi}"
+    elbow_joint_lower_limit="${-pi}" elbow_joint_upper_limit="${pi}"
     wrist_1_lower_limit="${-2*pi}" wrist_1_upper_limit="${2*pi}"
     wrist_2_lower_limit="${-2*pi}" wrist_2_upper_limit="${2*pi}"
@@ -27,5 +27,5 @@
   </xacro:sensor_d435>
   <xacro:sensor_d435 parent="world" name="camera_3_depth" topics_ns="camera_3_depth">
-    <origin xyz="0.7 0 1" rpy="0 ${pi/2} 0.0"/>
+    <origin xyz="0.7 0 0.65" rpy="0 ${pi/2} 0.0"/>
   </xacro:sensor_d435>
   <xacro:stereo_camera_v0 name="camera_1_stereo" image_format="R8G8B8"
@@ -42,6 +42,6 @@
   <xacro:stereo_camera_v0 name="camera_3_stereo" image_format="R8G8B8"
       parent="world" hfov="90" focal_length="639.997649"
-      image_width="1280" image_height="720">
-      <origin xyz="0.7 0 1" rpy="0 ${pi/2} 0" />
+      image_width="960" image_height="540">
+      <origin xyz="0.7 0 0.65" rpy="0 ${pi/2} 0" />
   </xacro:stereo_camera_v0>
   <link name="world" />

File: urdf/ur5_robotiq85_gripper.urdf.xacro (robot description, xacro)
@@ -31,6 +31,8 @@
   </joint>
   <gazebo reference="robotiq_coupler">
-    <mu1>0.9</mu1>
-    <mu2>0.9</mu2>
+    <kp>100000.0</kp>
+    <kd>1.0</kd>
+    <mu1>0.1</mu1>
+    <mu2>0.1</mu2>
     <material>Gazebo/FlatBlack</material>
   </gazebo>
